Commit message: double rotor and its plugin is added

File: vtol_description/urdf/vtol.urdf.xacro (robot description, xacro)
@@ -15,5 +15,5 @@
   <!-- Component versions -->
   <xacro:property name="base_version"    value="0_0_0"/>
-  <xacro:property name="rotor_type"    value="default"/>
+  <xacro:property name="rotor_type"    value="double"/>
   <xacro:property name="elevator_type"    value="default"/>
   <xacro:property name="aileron_type"    value="default"/>
