Commit message: wheels are added to description. And angle of attack code is added

File: vtol_description/urdf/aileron/default/aileron_parameters.urdf.xacro (robot description, xacro)
@@ -13,5 +13,5 @@
   <xacro:property name="x_aileron"   value= "-0.345"/> <!-- [m] -->
   <xacro:property name="y_aileron"   value= "0.59"/> <!-- [m] -->
-  <xacro:property name="z_aileron"   value= "0.05"/> <!-- [m] -->
+  <xacro:property name="z_aileron"   value= "-0.01"/> <!-- [m] -->
   <xacro:property name="yaw_aileron" value= "${PI*2/3-0.09}"/> <!-- [m] -->
 </robot>

File: vtol_description/urdf/base/0_0_0/vtol_base.urdf.xacro (robot description, xacro)
@@ -18,5 +18,5 @@
     <link name="${robot_name}_${name}">
       <visual>
-        <origin xyz="0 0 0" rpy="0 0 ${PI}"/>
+        <origin xyz="0 0 -0.05" rpy="0 0 ${PI}"/>
         <geometry>
           <!--box size="${L} ${W} ${H}" /-->
@@ -26,5 +26,5 @@
       </visual>
       <collision> <!-- Main Body -->
-        <origin xyz="-0.2 0 0" rpy="0 0 0"/>
+        <origin xyz="-0.2 0 -0.00" rpy="0 0 0"/>
         <geometry>
           <box size="${L} ${W} ${H}" />
@@ -48,4 +48,88 @@
       </inertial>
     </link>
+    <link name="${robot_name}_${name}_wheel_front">
+      <inertial>
+        <origin   xyz="0 0 0"
+                  rpy="0 0 0"/>
+        <mass     value="0.001"/>
+        <inertia  ixx="0.0000001" ixy="0.000" ixz="0.000"
+                  iyy="0.0000001" iyz="0.000" izz="0.0000001"/>
+      </inertial>
+      <visual>
+        <origin xyz="0 0 0" rpy="0 0 0"/>
+        <geometry>
+          <cylinder length="0.005" radius="0.03"/>
+        </geometry>
+        <material name="vtol_material" />
+      </visual>
+      <collision>
+        <origin xyz="0 0 0" rpy="0 0 0"/>
+        <geometry>
+          <cylinder length="0.005" radius="0.03"/>
+        </geometry>
+      </collision>
+    </link>
+    <joint name="${robot_name}_${name}_to_${name}_wheel_front" type="continuous">
+      <parent link="${robot_name}_${name}"/>
+      <child link="${robot_name}_${name}_wheel_front"/>
+      <origin xyz="0.1 0 -0.08 " rpy="${PI/2} 0 0"/>
+      <axis xyz="0 0 1" />
+    </joint>
+    <link name="${robot_name}_${name}_wheel_left_hind">
+      <inertial>
+        <origin   xyz="0 0 0"
+                  rpy="0 0 0"/>
+        <mass     value="0.001"/>
+        <inertia  ixx="0.0000001" ixy="0.000" ixz="0.000"
+                  iyy="0.0000001" iyz="0.000" izz="0.0000001"/>
+      </inertial>
+      <visual>
+        <origin xyz="0 0 0" rpy="0 0 0"/>
+        <geometry>
+          <cylinder length="0.005" radius="0.03"/>
+        </geometry>
+        <material name="vtol_material" />
+      </visual>
+      <collision>
+        <origin xyz="0 0 0" rpy="0 0 0"/>
+        <geometry>
+          <cylinder length="0.005" radius="0.03"/>
+        </geometry>
+      </collision>
+    </link>
+    <joint name="${robot_name}_${name}_to_${name}_wheel_left_hind" type="continuous">
+      <parent link="${robot_name}_${name}"/>
+      <child link="${robot_name}_${name}_wheel_left_hind"/>
+      <origin xyz="-0.1 -0.2 -0.08 " rpy="${PI/2} 0 0"/>
+      <axis xyz="0 0 1" />
+    </joint>
+    <link name="${robot_name}_${name}_wheel_right_hind">
+      <inertial>
+        <origin   xyz="0 0 0"
+                  rpy="0 0 0"/>
+        <mass     value="0.001"/>
+        <inertia  ixx="0.0000001" ixy="0.000" ixz="0.000"
+                  iyy="0.0000001" iyz="0.000" izz="0.0000001"/>
+      </inertial>
+      <visual>
+        <origin xyz="0 0 0" rpy="0 0 0"/>
+        <geometry>
+          <cylinder length="0.005" radius="0.03"/>
+        </geometry>
+        <material name="vtol_material" />
+      </visual>
+      <collision>
+        <origin xyz="0 0 0" rpy="0 0 0"/>
+        <geometry>
+          <cylinder length="0.005" radius="0.03"/>
+        </geometry>
+      </collision>
+    </link>
+    <joint name="${robot_name}_${name}_to_${name}_wheel_right_hind" type="continuous">
+      <parent link="${robot_name}_${name}"/>
+      <child link="${robot_name}_${name}_wheel_right_hind"/>
+      <origin xyz="-0.1 0.2 -0.08 " rpy="${PI/2} 0 0"/>
+      <axis xyz="0 0 1" />
+    </joint>
     <gazebo>
       <plugin name="gazebo_ros_control"

File: vtol_description/urdf/base/0_0_0/vtol_base_parameters.urdf.xacro (robot description, xacro)
@@ -10,4 +10,4 @@
   <xacro:property name="L"   value= "0.5"/> <!-- [m] -->
   <xacro:property name="W"   value= "1.5"/> <!-- [m] -->
-  <xacro:property name="H"   value= "0.2"/> <!-- [m] -->
+  <xacro:property name="H"   value= "0.1"/> <!-- [m] -->
 </robot>

File: vtol_description/urdf/elevator/default/elevator_parameters.urdf.xacro (robot description, xacro)
@@ -13,5 +13,5 @@
   <xacro:property name="x_elevator"   value= "-0.25"/> <!-- [m] -->
   <xacro:property name="y_elevator"   value= "0.38"/> <!-- [m] -->
-  <xacro:property name="z_elevator"   value= "0.05"/> <!-- [m] -->
+  <xacro:property name="z_elevator"   value= "-0.01"/> <!-- [m] -->
   <xacro:property name="yaw_elevator" value= "${PI*2/3-0.09}"/> <!-- [m] -->
 </robot>

File: vtol_description/urdf/rotor/double/front_rotor_parameters.urdf.xacro (robot description, xacro)
@@ -19,5 +19,5 @@
   <xacro:property name="x_rotor"   value= "0.15"/> <!-- [m] -->
   <xacro:property name="y_rotor"   value= "0.25"/> <!-- [m] -->
-  <xacro:property name="z_rotor"   value= "0.1"/> <!-- [m] -->
+  <xacro:property name="z_rotor"   value= "0.05"/> <!-- [m] -->
   <xacro:property name="r_blade"   value= "0.1"/> <!-- [m] -->
   <xacro:property name="w_blade"   value= "0.02"/> <!-- [m] -->

File: vtol_description/urdf/rotor/double/hind_rotor_parameters.urdf.xacro (robot description, xacro)
@@ -19,5 +19,5 @@
   <xacro:property name="x_rotor"   value= "0.4"/> <!-- [m] -->
   <xacro:property name="y_rotor"   value= "0.0"/> <!-- [m] -->
-  <xacro:property name="z_rotor"   value= "0.1"/> <!-- [m] -->
+  <xacro:property name="z_rotor"   value= "0.05"/> <!-- [m] -->
   <xacro:property name="r_blade"   value= "0.1"/> <!-- [m] -->
   <xacro:property name="w_blade"   value= "0.02"/> <!-- [m] -->
